File: L000-Power/L000-Power-Schematic.sch (EAGLE design)
At the start: 59 parts, among them IC1 LM7805, IC2 LM7905, IC3 LM7809, IC4 LM7909, X1 JST-XH-2PIN, X10 JST-XH-5PIN, X11 JST-XH-5PIN, X12 JST-XH-5PIN, X13 JST-XH-5PIN, X14 JST-XH-5PIN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

Commit message: Update Power Schematic
Missing Juctions
Connections:
- net 5V+: now also X10.2, X11.2, X2.2, X3.2, X4.2, X5.2, X6.2, X7.2, X8.2, X9.2
- net 5V-: now also X10.1, X2.1, X3.1, X4.1, X5.1, X6.1, X7.1, X8.1, X9.1
- net 9V+: now also X10.4, X2.4, X3.4, X4.4, X5.4, X6.4, X7.4, X8.4, X9.4
- net 9V-: now also X10.3, X11.3, X2.3, X3.3, X4.3, X5.3, X6.3, X7.3, X8.3, X9.3
- net GND: now also X10.5, X11.5, X2.5, X3.5, X4.5, X5.5, X6.5, X7.5, X8.5, X9.5
Changed lines of the file:
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@@
 </segment>
 <segment>
-<wire x1="121.92" y1="-129.54" x2="2.54" y2="-129.54" width="0.1524" layer="91"/>
+<wire x1="121.92" y1="-129.54" x2="119.38" y2="-129.54" width="0.1524" layer="91"/>
 <label x="-2.54" y="-129.54" size="1.778" layer="95"/>
+<pinref part="X2" gate="G$1" pin="5"/>
+<junction x="5.08" y="-129.54"/>
+<wire x1="119.38" y1="-129.54" x2="106.68" y2="-129.54" width="0.1524" layer="91"/>
+<wire x1="106.68" y1="-129.54" x2="93.98" y2="-129.54" width="0.1524" layer="91"/>
+<wire x1="93.98" y1="-129.54" x2="81.28" y2="-129.54" width="0.1524" layer="91"/>
+<wire x1="81.28" y1="-129.54" x2="68.58" y2="-129.54" width="0.1524" layer="91"/>
+<wire x1="68.58" y1="-129.54" x2="55.88" y2="-129.54" width="0.1524" layer="91"/>
+<wire x1="55.88" y1="-129.54" x2="43.18" y2="-129.54" width="0.1524" layer="91"/>
+<wire x1="43.18" y1="-129.54" x2="30.48" y2="-129.54" width="0.1524" layer="91"/>
+<wire x1="30.48" y1="-129.54" x2="17.78" y2="-129.54" width="0.1524" layer="91"/>
+<wire x1="17.78" y1="-129.54" x2="5.08" y2="-129.54" width="0.1524" layer="91"/>
+<wire x1="5.08" y1="-129.54" x2="2.54" y2="-129.54" width="0.1524" layer="91"/>
+<pinref part="X3" gate="G$1" pin="5"/>
+<junction x="17.78" y="-129.54"/>
+<pinref part="X4" gate="G$1" pin="5"/>
+<junction x="30.48" y="-129.54"/>
+<pinref part="X5" gate="G$1" pin="5"/>
+<junction x="43.18" y="-129.54"/>
+<pinref part="X6" gate="G$1" pin="5"/>
+<junction x="55.88" y="-129.54"/>
+<pinref part="X7" gate="G$1" pin="5"/>
+<junction x="68.58" y="-129.54"/>
+<pinref part="X8" gate="G$1" pin="5"/>
+<junction x="81.28" y="-129.54"/>
+<pinref part="X9" gate="G$1" pin="5"/>
+<junction x="93.98" y="-129.54"/>
+<pinref part="X10" gate="G$1" pin="5"/>
+<junction x="106.68" y="-129.54"/>
+<pinref part="X11" gate="G$1" pin="5"/>
+<junction x="119.38" y="-129.54"/>
 </segment>
 <segment>
@@
 </segment>
 <segment>
-<wire x1="121.92" y1="-121.92" x2="2.54" y2="-121.92" width="0.1524" layer="91"/>
+<wire x1="121.92" y1="-121.92" x2="119.38" y2="-121.92" width="0.1524" layer="91"/>
 <label x="-2.54" y="-121.92" size="1.778" layer="95"/>
+<pinref part="X2" gate="G$1" pin="2"/>
+<junction x="5.08" y="-121.92"/>
+<wire x1="119.38" y1="-121.92" x2="106.68" y2="-121.92" width="0.1524" layer="91"/>
+<wire x1="106.68" y1="-121.92" x2="93.98" y2="-121.92" width="0.1524" layer="91"/>
+<wire x1="93.98" y1="-121.92" x2="81.28" y2="-121.92" width="0.1524" layer="91"/>
+<wire x1="81.28" y1="-121.92" x2="68.58" y2="-121.92" width="0.1524" layer="91"/>
+<wire x1="68.58" y1="-121.92" x2="55.88" y2="-121.92" width="0.1524" layer="91"/>
+<wire x1="55.88" y1="-121.92" x2="43.18" y2="-121.92" width="0.1524" layer="91"/>
+<wire x1="43.18" y1="-121.92" x2="30.48" y2="-121.92" width="0.1524" layer="91"/>
+<wire x1="30.48" y1="-121.92" x2="17.78" y2="-121.92" width="0.1524" layer="91"/>
+<wire x1="17.78" y1="-121.92" x2="5.08" y2="-121.92" width="0.1524" layer="91"/>
+<wire x1="5.08" y1="-121.92" x2="2.54" y2="-121.92" width="0.1524" layer="91"/>
+<pinref part="X3" gate="G$1" pin="2"/>
+<junction x="17.78" y="-121.92"/>
+<pinref part="X4" gate="G$1" pin="2"/>
+<junction x="30.48" y="-121.92"/>
+<pinref part="X5" gate="G$1" pin="2"/>
+<junction x="43.18" y="-121.92"/>
+<pinref part="X6" gate="G$1" pin="2"/>
+<junction x="55.88" y="-121.92"/>
+<pinref part="X7" gate="G$1" pin="2"/>
+<junction x="68.58" y="-121.92"/>
+<pinref part="X8" gate="G$1" pin="2"/>
+<junction x="81.28" y="-121.92"/>
+<pinref part="X9" gate="G$1" pin="2"/>
+<junction x="93.98" y="-121.92"/>
+<pinref part="X10" gate="G$1" pin="2"/>
+<junction x="106.68" y="-121.92"/>
+<pinref part="X11" gate="G$1" pin="2"/>
+<junction x="119.38" y="-121.92"/>
 </segment>
 <segment>
@@
 <segment>
 <pinref part="X11" gate="G$1" pin="1"/>
-<wire x1="119.38" y1="-119.38" x2="2.54" y2="-119.38" width="0.1524" layer="91"/>
+<wire x1="119.38" y1="-119.38" x2="106.68" y2="-119.38" width="0.1524" layer="91"/>
 <label x="-2.54" y="-119.38" size="1.778" layer="95"/>
+<pinref part="X2" gate="G$1" pin="1"/>
+<junction x="5.08" y="-119.38"/>
+<wire x1="106.68" y1="-119.38" x2="93.98" y2="-119.38" width="0.1524" layer="91"/>
+<wire x1="93.98" y1="-119.38" x2="81.28" y2="-119.38" width="0.1524" layer="91"/>
+<wire x1="81.28" y1="-119.38" x2="68.58" y2="-119.38" width="0.1524" layer="91"/>
+<wire x1="68.58" y1="-119.38" x2="55.88" y2="-119.38" width="0.1524" layer="91"/>
+<wire x1="55.88" y1="-119.38" x2="43.18" y2="-119.38" width="0.1524" layer="91"/>
+<wire x1="43.18" y1="-119.38" x2="30.48" y2="-119.38" width="0.1524" layer="91"/>
+<wire x1="30.48" y1="-119.38" x2="17.78" y2="-119.38" width="0.1524" layer="91"/>
+<wire x1="17.78" y1="-119.38" x2="5.08" y2="-119.38" width="0.1524" layer="91"/>
+<wire x1="5.08" y1="-119.38" x2="2.54" y2="-119.38" width="0.1524" layer="91"/>
+<pinref part="X3" gate="G$1" pin="1"/>
+<junction x="17.78" y="-119.38"/>
+<pinref part="X4" gate="G$1" pin="1"/>
+<junction x="30.48" y="-119.38"/>
+<pinref part="X5" gate="G$1" pin="1"/>
+<junction x="43.18" y="-119.38"/>
+<pinref part="X6" gate="G$1" pin="1"/>
+<junction x="55.88" y="-119.38"/>
+<pinref part="X7" gate="G$1" pin="1"/>
+<junction x="68.58" y="-119.38"/>
+<pinref part="X8" gate="G$1" pin="1"/>
+<junction x="81.28" y="-119.38"/>
+<pinref part="X9" gate="G$1" pin="1"/>
+<junction x="93.98" y="-119.38"/>
+<pinref part="X10" gate="G$1" pin="1"/>
+<junction x="106.68" y="-119.38"/>
+<junction x="119.38" y="-119.38"/>
 </segment>
 <segment>
@@
 <pinref part="X20" gate="G$1" pin="1"/>
 <junction x="106.68" y="-142.24"/>
+<junction x="119.38" y="-142.24"/>
 </segment>
 </net>
@@
 <segment>
 <pinref part="X11" gate="G$1" pin="4"/>
-<wire x1="119.38" y1="-127" x2="2.54" y2="-127" width="0.1524" layer="91"/>
+<wire x1="119.38" y1="-127" x2="106.68" y2="-127" width="0.1524" layer="91"/>
 <label x="-2.54" y="-127" size="1.778" layer="95"/>
+<pinref part="X2" gate="G$1" pin="4"/>
+<junction x="5.08" y="-127"/>
+<wire x1="106.68" y1="-127" x2="93.98" y2="-127" width="0.1524" layer="91"/>
+<wire x1="93.98" y1="-127" x2="81.28" y2="-127" width="0.1524" layer="91"/>
+<wire x1="81.28" y1="-127" x2="68.58" y2="-127" width="0.1524" layer="91"/>
+<wire x1="68.58" y1="-127" x2="55.88" y2="-127" width="0.1524" layer="91"/>
+<wire x1="55.88" y1="-127" x2="43.18" y2="-127" width="0.1524" layer="91"/>
+<wire x1="43.18" y1="-127" x2="30.48" y2="-127" width="0.1524" layer="91"/>
+<wire x1="30.48" y1="-127" x2="17.78" y2="-127" width="0.1524" layer="91"/>
+<wire x1="17.78" y1="-127" x2="5.08" y2="-127" width="0.1524" layer="91"/>
+<wire x1="5.08" y1="-127" x2="2.54" y2="-127" width="0.1524" layer="91"/>
+<pinref part="X3" gate="G$1" pin="4"/>
+<junction x="17.78" y="-127"/>
+<pinref part="X4" gate="G$1" pin="4"/>
+<junction x="30.48" y="-127"/>
+<pinref part="X5" gate="G$1" pin="4"/>
+<junction x="43.18" y="-127"/>
+<pinref part="X6" gate="G$1" pin="4"/>
+<junction x="55.88" y="-127"/>
+<pinref part="X7" gate="G$1" pin="4"/>
+<junction x="68.58" y="-127"/>
+<pinref part="X8" gate="G$1" pin="4"/>
+<junction x="81.28" y="-127"/>
+<pinref part="X9" gate="G$1" pin="4"/>
+<junction x="93.98" y="-127"/>
+<pinref part="X10" gate="G$1" pin="4"/>
+<junction x="106.68" y="-127"/>
+<junction x="119.38" y="-127"/>
 </segment>
 <segment>
@@
 <pinref part="X20" gate="G$1" pin="4"/>
 <junction x="106.68" y="-149.86"/>
+<junction x="119.38" y="-149.86"/>
 </segment>
 </net>
@@
 </segment>
 <segment>
-<wire x1="121.92" y1="-124.46" x2="2.54" y2="-124.46" width="0.1524" layer="91"/>
+<wire x1="121.92" y1="-124.46" x2="119.38" y2="-124.46" width="0.1524" layer="91"/>
 <label x="-2.54" y="-124.46" size="1.778" layer="95"/>
+<pinref part="X2" gate="G$1" pin="3"/>
+<junction x="5.08" y="-124.46"/>
+<wire x1="119.38" y1="-124.46" x2="106.68" y2="-124.46" width="0.1524" layer="91"/>
+<wire x1="106.68" y1="-124.46" x2="93.98" y2="-124.46" width="0.1524" layer="91"/>
+<wire x1="93.98" y1="-124.46" x2="81.28" y2="-124.46" width="0.1524" layer="91"/>
+<wire x1="81.28" y1="-124.46" x2="68.58" y2="-124.46" width="0.1524" layer="91"/>
+<wire x1="68.58" y1="-124.46" x2="55.88" y2="-124.46" width="0.1524" layer="91"/>
+<wire x1="55.88" y1="-124.46" x2="43.18" y2="-124.46" width="0.1524" layer="91"/>
+<wire x1="43.18" y1="-124.46" x2="30.48" y2="-124.46" width="0.1524" layer="91"/>
+<wire x1="30.48" y1="-124.46" x2="17.78" y2="-124.46" width="0.1524" layer="91"/>
+<wire x1="17.78" y1="-124.46" x2="5.08" y2="-124.46" width="0.1524" layer="91"/>
+<wire x1="5.08" y1="-124.46" x2="2.54" y2="-124.46" width="0.1524" layer="91"/>
+<pinref part="X3" gate="G$1" pin="3"/>
+<junction x="17.78" y="-124.46"/>
+<pinref part="X4" gate="G$1" pin="3"/>
+<junction x="30.48" y="-124.46"/>
+<pinref part="X5" gate="G$1" pin="3"/>
+<junction x="43.18" y="-124.46"/>
+<pinref part="X6" gate="G$1" pin="3"/>
+<junction x="55.88" y="-124.46"/>
+<pinref part="X7" gate="G$1" pin="3"/>
+<junction x="68.58" y="-124.46"/>
+<pinref part="X8" gate="G$1" pin="3"/>
+<junction x="81.28" y="-124.46"/>
+<pinref part="X9" gate="G$1" pin="3"/>
+<junction x="93.98" y="-124.46"/>
+<pinref part="X10" gate="G$1" pin="3"/>
+<junction x="106.68" y="-124.46"/>
+<pinref part="X11" gate="G$1" pin="3"/>
+<junction x="119.38" y="-124.46"/>
 </segment>
 <segment>
@@
 </sheet>
 </sheets>
-<errors>
-</errors>
 </schematic>
 </drawing>
