File: L000-Power/L000-Power-Schematic.sch (EAGLE design)
At the start: 61 parts, among them X1 JST-XH-2PIN, X10 JST-XH-5PIN, X11 JST-XH-5PIN, X12 JST-XH-5PIN, X13 JST-XH-5PIN, X14 JST-XH-5PIN, X15 JST-XH-5PIN, X16 JST-XH-5PIN, X17 JST-XH-5PIN, X18 JST-XH-5PIN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

Commit message: Fixes
Parts:
- R10, R9: value 220K -> ?
- R11, R12: value 120K -> ?
Changed lines of the file:
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@@
 <part name="LED1" library="led" deviceset="LED" device="5MM"/>
 <part name="LED2" library="led" deviceset="LED" device="5MM"/>
-<part name="R11" library="resistor" deviceset="R-US_" device="0309/10" value="120K"/>
-<part name="R12" library="resistor" deviceset="R-US_" device="0309/10" value="120K"/>
-<part name="R9" library="resistor" deviceset="R-US_" device="0309/10" value="220K"/>
-<part name="R10" library="resistor" deviceset="R-US_" device="0309/10" value="220K"/>
+<part name="R11" library="resistor" deviceset="R-US_" device="0309/10" value="?"/>
+<part name="R12" library="resistor" deviceset="R-US_" device="0309/10" value="?"/>
+<part name="R9" library="resistor" deviceset="R-US_" device="0309/10" value="?"/>
+<part name="R10" library="resistor" deviceset="R-US_" device="0309/10" value="?"/>
 </parts>
 <sheets>

Commit message: Normalize all output resistor to 10k
Parts:
- R10, R9: value ? -> 2K
- R11, R12: value ? -> 1K
Changed lines of the file:
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@@
 <part name="LED1" library="led" deviceset="LED" device="5MM"/>
 <part name="LED2" library="led" deviceset="LED" device="5MM"/>
-<part name="R11" library="resistor" deviceset="R-US_" device="0309/10" value="?"/>
-<part name="R12" library="resistor" deviceset="R-US_" device="0309/10" value="?"/>
-<part name="R9" library="resistor" deviceset="R-US_" device="0309/10" value="?"/>
-<part name="R10" library="resistor" deviceset="R-US_" device="0309/10" value="?"/>
+<part name="R11" library="resistor" deviceset="R-US_" device="0309/10" value="1K"/>
+<part name="R12" library="resistor" deviceset="R-US_" device="0309/10" value="1K"/>
+<part name="R9" library="resistor" deviceset="R-US_" device="0309/10" value="2K"/>
+<part name="R10" library="resistor" deviceset="R-US_" device="0309/10" value="2K"/>
 </parts>
 <sheets>
