File: L002-Square/L002 - Square - Schematic.sch (EAGLE design)
At the start: 11 parts, among them IC1 40106, Q1 2N3906

Commit message: Fixes
Parts:
- removed Q1: 2N3906, transistor-pnp:2N3906
- removed R3: 10k, resistor:R-US_VMTA55
- added C2: 0.1~1uF, rcl:CPOL-USE2.5-6
- R1: value 4.7K -> 2~4K
- R4: value 120K -> 4.7K
- R5: value 10K -> 1K
Connections:
- removed net N$4: Q1.E, R4.1
- removed net N$5: Q1.B, R3.1
- removed net N$6: D1.A, R4.2
- new net N$3: D1.A, R4.1
- net 5V+: now also C2.+; no longer D1.C
- net 5V-: now also C2.-, D1.C; no longer Q1.C
- net OUTPUT: now also R4.2; no longer R3.2
Other:
- note added: "close to 40106 power pins."
- note added: "this x6"
- moved on the sheet: D1, D2, D3, R4, R5
Changed lines of the file:
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@@
 <parts>
 <part name="IC1" library="40xx" deviceset="40106" device="N" value="40106"/>
-<part name="R1" library="resistor" deviceset="R-US_" device="VMTA55" value="4.7K"/>
+<part name="R1" library="resistor" deviceset="R-US_" device="VMTA55" value="2~4K"/>
 <part name="C1" library="rcl" deviceset="CPOL-US" device="E2.5-6" value="1uF"/>
 <part name="R2" library="pot" deviceset="US-EVU" device="M" technology="F3" value="1M"/>
-<part name="Q1" library="transistor-pnp" deviceset="2N3906" device=""/>
-<part name="R3" library="resistor" deviceset="R-US_" device="VMTA55" value="10k"/>
-<part name="R4" library="resistor" deviceset="R-US_" device="VMTA55" value="120K"/>
+<part name="R4" library="resistor" deviceset="R-US_" device="VMTA55" value="4.7K"/>
 <part name="D1" library="led" deviceset="SFH482" device="" value="LED"/>
 <part name="D2" library="diode" deviceset="1N581*" device="" technology="7-B" value="1N5817"/>
 <part name="D3" library="diode" deviceset="1N581*" device="" technology="7-B" value="1N5817"/>
-<part name="R5" library="resistor" deviceset="R-US_" device="VMTA55" value="10K"/>
+<part name="R5" library="resistor" deviceset="R-US_" device="VMTA55" value="1K"/>
+<part name="C2" library="rcl" deviceset="CPOL-US" device="E2.5-6" value="0.1~1uF"/>
 </parts>
 <sheets>
 <sheet>
 <plain>
+<text x="27.94" y="40.64" size="1.778" layer="91">this x6</text>
+<text x="63.5" y="99.06" size="1.778" layer="91">close to 40106 power pins.</text>
 </plain>
 <instances>
@@
 <instance part="C1" gate="G$1" x="10.16" y="50.8"/>
 <instance part="R2" gate="G$1" x="25.4" y="71.12" rot="R90"/>
-<instance part="Q1" gate="G$1" x="53.34" y="71.12"/>
-<instance part="R3" gate="G$1" x="45.72" y="71.12" rot="R180"/>
-<instance part="R4" gate="G$1" x="55.88" y="81.28" rot="R90"/>
-<instance part="D1" gate="1" x="55.88" y="88.9" rot="R180"/>
-<instance part="D2" gate="G$1" x="66.04" y="60.96" rot="R90"/>
-<instance part="D3" gate="G$1" x="66.04" y="48.26" rot="R90"/>
-<instance part="R5" gate="G$1" x="73.66" y="55.88" rot="R180"/>
+<instance part="R4" gate="G$1" x="50.8" y="48.26" rot="R90"/>
+<instance part="D1" gate="1" x="50.8" y="38.1"/>
+<instance part="D2" gate="G$1" x="60.96" y="60.96" rot="R90"/>
+<instance part="D3" gate="G$1" x="60.96" y="50.8" rot="R90"/>
+<instance part="R5" gate="G$1" x="71.12" y="55.88" rot="R180"/>
+<instance part="C2" gate="G$1" x="83.82" y="91.44"/>
 </instances>
 <busses>
@@
 <wire x1="33.02" y1="78.74" x2="33.02" y2="71.12" width="0.1524" layer="91"/>
 <junction x="33.02" y="71.12"/>
-<pinref part="R3" gate="G$1" pin="2"/>
 <wire x1="40.64" y1="71.12" x2="40.64" y2="55.88" width="0.1524" layer="91"/>
+<junction x="40.64" y="55.88"/>
+<pinref part="D3" gate="G$1" pin="C"/>
 <pinref part="D2" gate="G$1" pin="A"/>
-<pinref part="D3" gate="G$1" pin="C"/>
-<wire x1="66.04" y1="58.42" x2="66.04" y2="55.88" width="0.1524" layer="91"/>
+<wire x1="60.96" y1="58.42" x2="60.96" y2="55.88" width="0.1524" layer="91"/>
+<wire x1="60.96" y1="55.88" x2="60.96" y2="53.34" width="0.1524" layer="91"/>
 <pinref part="R5" gate="G$1" pin="2"/>
-<wire x1="66.04" y1="55.88" x2="66.04" y2="50.8" width="0.1524" layer="91"/>
-<wire x1="68.58" y1="55.88" x2="66.04" y2="55.88" width="0.1524" layer="91"/>
-<junction x="66.04" y="55.88"/>
-<wire x1="66.04" y1="55.88" x2="40.64" y2="55.88" width="0.1524" layer="91"/>
-<junction x="40.64" y="55.88"/>
+<wire x1="66.04" y1="55.88" x2="60.96" y2="55.88" width="0.1524" layer="91"/>
+<junction x="60.96" y="55.88"/>
+<wire x1="40.64" y1="55.88" x2="50.8" y2="55.88" width="0.1524" layer="91"/>
+<pinref part="R4" gate="G$1" pin="2"/>
+<wire x1="50.8" y1="55.88" x2="60.96" y2="55.88" width="0.1524" layer="91"/>
+<wire x1="50.8" y1="53.34" x2="50.8" y2="55.88" width="0.1524" layer="91"/>
+<junction x="50.8" y="55.88"/>
 </segment>
 <segment>
 <pinref part="R5" gate="G$1" pin="1"/>
-<wire x1="78.74" y1="55.88" x2="81.28" y2="55.88" width="0.1524" layer="91"/>
+<wire x1="76.2" y1="55.88" x2="78.74" y2="55.88" width="0.1524" layer="91"/>
 <label x="81.28" y="55.88" size="1.778" layer="95"/>
 </segment>
@@
 <pinref part="C1" gate="G$1" pin="-"/>
 <wire x1="10.16" y1="45.72" x2="10.16" y2="43.18" width="0.1524" layer="91"/>
-<label x="10.16" y="43.18" size="1.778" layer="95"/>
-</segment>
-<segment>
-<pinref part="Q1" gate="G$1" pin="C"/>
-<wire x1="55.88" y1="66.04" x2="55.88" y2="63.5" width="0.1524" layer="91"/>
-<label x="55.88" y="63.5" size="1.778" layer="95"/>
+<label x="10.16" y="40.64" size="1.778" layer="95"/>
 </segment>
 <segment>
 <pinref part="D3" gate="G$1" pin="A"/>
-<wire x1="66.04" y1="45.72" x2="66.04" y2="43.18" width="0.1524" layer="91"/>
-<label x="66.04" y="40.64" size="1.778" layer="95"/>
+<wire x1="60.96" y1="48.26" x2="60.96" y2="43.18" width="0.1524" layer="91"/>
+<label x="60.96" y="40.64" size="1.778" layer="95"/>
 </segment>
-</net>
-<net name="N$4" class="0">
 <segment>
-<pinref part="Q1" gate="G$1" pin="E"/>
-<pinref part="R4" gate="G$1" pin="1"/>
+<pinref part="D1" gate="1" pin="C"/>
+<wire x1="50.8" y1="33.02" x2="50.8" y2="30.48" width="0.1524" layer="91"/>
+<label x="50.8" y="27.94" size="1.778" layer="95"/>
 </segment>
-</net>
-<net name="N$5" class="0">
 <segment>
-<pinref part="Q1" gate="G$1" pin="B"/>
-<pinref part="R3" gate="G$1" pin="1"/>
-</segment>
-</net>
-<net name="N$6" class="0">
-<segment>
-<pinref part="R4" gate="G$1" pin="2"/>
-<pinref part="D1" gate="1" pin="A"/>
+<wire x1="76.2" y1="83.82" x2="83.82" y2="83.82" width="0.1524" layer="91"/>
+<label x="71.12" y="83.82" size="1.778" layer="95"/>
+<pinref part="C2" gate="G$1" pin="-"/>
+<wire x1="83.82" y1="86.36" x2="83.82" y2="83.82" width="0.1524" layer="91"/>
+<wire x1="83.82" y1="83.82" x2="91.44" y2="83.82" width="0.1524" layer="91"/>
+<junction x="83.82" y="83.82"/>
 </segment>
 </net>
 <net name="5V+" class="0">
 <segment>
-<pinref part="D1" gate="1" pin="C"/>
-<wire x1="55.88" y1="93.98" x2="55.88" y2="96.52" width="0.1524" layer="91"/>
-<label x="55.88" y="96.52" size="1.778" layer="95"/>
+<pinref part="D2" gate="G$1" pin="C"/>
+<wire x1="60.96" y1="63.5" x2="60.96" y2="68.58" width="0.1524" layer="91"/>
+<label x="60.96" y="68.58" size="1.778" layer="95"/>
 </segment>
 <segment>
-<pinref part="D2" gate="G$1" pin="C"/>
-<wire x1="66.04" y1="63.5" x2="66.04" y2="66.04" width="0.1524" layer="91"/>
-<label x="66.04" y="68.58" size="1.778" layer="95"/>
+<wire x1="76.2" y1="96.52" x2="83.82" y2="96.52" width="0.1524" layer="91"/>
+<label x="71.12" y="93.98" size="1.778" layer="95"/>
+<pinref part="C2" gate="G$1" pin="+"/>
+<wire x1="83.82" y1="96.52" x2="83.82" y2="93.98" width="0.1524" layer="91"/>
+<wire x1="83.82" y1="96.52" x2="91.44" y2="96.52" width="0.1524" layer="91"/>
+<junction x="83.82" y="96.52"/>
 </segment>
 </net>
+<net name="N$3" class="0">
+<segment>
+<pinref part="R4" gate="G$1" pin="1"/>
+<pinref part="D1" gate="1" pin="A"/>
+<wire x1="50.8" y1="43.18" x2="50.8" y2="40.64" width="0.1524" layer="91"/>
+</segment>
+</net>
