File: L002-Square/L002 - Square - Schematic.sch (EAGLE design)
At the start: 10 parts, among them IC1 40106

Commit message: Update everything to use 1n60p Schottky diodes
Parts:
- D2, D3: value 1N5817 -> 1N60P
Changed lines of the file:
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@@
 <part name="R4" library="resistor" deviceset="R-US_" device="VMTA55" value="4.7K"/>
 <part name="D1" library="led" deviceset="SFH482" device="" value="LED"/>
-<part name="D2" library="diode" deviceset="1N581*" device="" technology="7-B" value="1N5817"/>
-<part name="D3" library="diode" deviceset="1N581*" device="" technology="7-B" value="1N5817"/>
+<part name="D2" library="diode" deviceset="1N581*" device="" technology="7-B" value="1N60P"/>
+<part name="D3" library="diode" deviceset="1N581*" device="" technology="7-B" value="1N60P"/>
 <part name="R5" library="resistor" deviceset="R-US_" device="VMTA55" value="1K"/>
 <part name="C2" library="rcl" deviceset="CPOL-US" device="E2.5-6" value="0.1~1uF"/>

Commit message: 10k r on outputs
Parts:
- R5: value 1K -> 10K
Changed lines of the file:
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@@
 <part name="D2" library="diode" deviceset="1N581*" device="" technology="7-B" value="1N60P"/>
 <part name="D3" library="diode" deviceset="1N581*" device="" technology="7-B" value="1N60P"/>
-<part name="R5" library="resistor" deviceset="R-US_" device="VMTA55" value="1K"/>
+<part name="R5" library="resistor" deviceset="R-US_" device="VMTA55" value="10K"/>
 <part name="C2" library="rcl" deviceset="CPOL-US" device="E2.5-6" value="0.1~1uF"/>
 </parts>

Commit message: Updated strip boards
Parts:
- R1: value 2~4K -> 4.7K
Changed lines of the file:
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@@
 <parts>
 <part name="IC1" library="40xx" deviceset="40106" device="N" value="40106"/>
-<part name="R1" library="resistor" deviceset="R-US_" device="VMTA55" value="2~4K"/>
+<part name="R1" library="resistor" deviceset="R-US_" device="VMTA55" value="4.7K"/>
 <part name="C1" library="rcl" deviceset="CPOL-US" device="E2.5-6" value="1uF"/>
 <part name="R2" library="pot" deviceset="US-EVU" device="M" technology="F3" value="1M"/>
